File: Torturous/Torturous.kicad_sch (KiCad schematic)
At the start: 40 parts, among them U2 nice_nano

Commit message: finnished v0.1 schematics
Parts:
- added D20: 1N4148W, Diode_SMD:D_SOD-123, symbol Diode:1N4148W
- added J1: Conn_01x04_Pin, symbol Connector:Conn_01x04_Pin
- added J4: Conn_01x08_Pin, symbol Connector:Conn_01x08_Pin
- added S1: 463091370402, 463091370402:463091370402, symbol Micro Switch:463091370402
- added SW1: RotaryEncoder, symbol Device:RotaryEncoder
Connections:
- net COL5: now also S1.1
- net ROW3: now also J4.6 (Pin_6)
- net ROW4: now also D20.1 (K), J1.1 (Pin_1)
- net ROTa: now reaches U2.11 (P1.04-LF)
- net ROTa: now also SW1.A
- net ROTb: now reaches U2.12 (P1.06-LF)
- net ROTb: now also SW1.B
- net at U2.16 (3V3): now also J4.1 (Pin_1)
- net at U2.17 (P0.31-LF): now also J4.3 (Pin_3)
- net at U2.18 (P0.29-LF): now also J4.4 (Pin_4)
- net at U2.20 (P1.15-LF): now also J4.5 (Pin_5)
- net COL6: now reaches U2.21 (P1.13-LF)
- net COL6: now also J1.2 (Pin_2), J4.7 (Pin_7)
- new net: D20.2 (A), S1.2
- new net GND: J4.2 (Pin_2), SW1.C
Other:
- added sheet HE (he.kicad_sch)
- added sheet Thumb (thumb.kicad_sch)
- note added: "0.1"
- note added: "05.07.2026"
- note added: "Main board"
