File: Torturous/Torturous.kicad_sch (KiCad schematic)
At the start: 45 parts, among them J1 Conn_01x04_Pin, J4 Conn_01x08_Pin, SW1 RotaryEncoder, U2 nice_nano

Commit message: started the phys layout
Parts:
- BT1: footprint (none) -> Connector_JST:JST_PH_S2B-PH-K_1x02_P2.00mm_Horizontal
- J1: footprint (none) -> Connector_FFC-FPC:Amphenol_F32Q-1A7x1-11004_1x04-1MP_P0.5mm_Horizontal
- J4: footprint (none) -> Connector_FFC-FPC:Hirose_FH12-8S-0.5SH_1x08-1MP_P0.50mm_Horizontal
- S1: footprint 463091370402:463091370402 -> Microswith:463091370402
- SW1: footprint (none) -> Connector_PinHeader_2.54mm:PinHeader_1x03_P2.54mm_Vertical
Changed lines of the file:
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@@
 			)
 		)
-		(property "Footprint" ""
+		(property "Footprint" "Connector_JST:JST_PH_S2B-PH-K_1x02_P2.00mm_Horizontal"
 			(at 84.836 34.29 90)
 			(hide yes)
@@
 			)
 		)
-		(property "Footprint" ""
+		(property "Footprint" "Connector_FFC-FPC:Amphenol_F32Q-1A7x1-11004_1x04-1MP_P0.5mm_Horizontal"
 			(at 80.01 176.53 0)
 			(hide yes)
@@
 			)
 		)
-		(property "Footprint" "463091370402:463091370402"
+		(property "Footprint" "Microswith:463091370402"
 			(at 115.57 156.21 0)
 			(hide yes)
@@
 			)
 		)
-		(property "Footprint" ""
+		(property "Footprint" "Connector_PinHeader_2.54mm:PinHeader_1x03_P2.54mm_Vertical"
 			(at 129.794 138.43 0)
 			(hide yes)
@@
 			)
 		)
-		(property "Footprint" ""
+		(property "Footprint" "Connector_FFC-FPC:Hirose_FH12-8S-0.5SH_1x08-1MP_P0.50mm_Horizontal"
 			(at 110.49 52.07 0)
 			(hide yes)

Commit message: routing finnished for the main board
Parts:
- removed MX1, MX10, MX11, MX12, MX13, MX14, MX15, MX16, MX17, MX18, MX19, MX2, MX3, MX4, MX5, MX6, MX7, MX8, MX9: MX_SW_solder, PCM_marbastlib-mx:SW_MX_1u, symbol PCM_marbastlib-mx:MX_SW_solder
- added MX1, MX10, MX11, MX12, MX13, MX14, MX15, MX16, MX17, MX18, MX19, MX2, MX3, MX4, MX5, MX6, MX7, MX8, MX9: MX_SW_HS, PCM_marbastlib-mx:SW_MX_HS_CPG151101S11_1u, symbol PCM_marbastlib-mx:MX_SW_HS_CPG151101S11
Connections:
- net COL1: now also MX1.1, MX11.1, MX16.1, MX6.1
- net COL2: now also MX12.1, MX17.1, MX2.1, MX7.1
- net COL3: now also MX13.1, MX18.1, MX3.1, MX8.1
- net COL4: now also MX14.1, MX19.1, MX4.1, MX9.1
- net COL5: now also MX10.1, MX15.1, MX5.1
- net ROW1: now also U2.5 (P0.17); no longer U2.8 (P0.24)
- net ROW2: now also U2.6 (P0.20); no longer U2.7 (P0.22)
- net ROW3: now also U2.7 (P0.22); no longer U2.6 (P0.20)
- net ROW4: now also U2.8 (P0.24); no longer U2.5 (P0.17)
- net at D8.2 (A): now also MX14.2
- net at D2.2 (A): now also MX17.2
- net at D9.2 (A): now also MX15.2
- net at D14.2 (A): now also MX10.2
- net at D11.2 (A): now also MX7.2
- net at D1.2 (A): now also MX16.2
- net J4 PIN3: now reaches J4.3 (Pin_3)
- net J4 PIN3: now also U2.20 (P1.15-LF); no longer U2.17 (P0.31-LF)
- net J4 PIN4: now reaches J4.4 (Pin_4), U2.18 (P0.29-LF)
- net J4 PIN5: now reaches J4.5 (Pin_5)
- net J4 PIN5: now also U2.17 (P0.31-LF); no longer U2.20 (P1.15-LF)
- net at D13.2 (A): now also MX9.2
- net at D4.2 (A): now also MX19.2
- net at D18.2 (A): now also MX4.2
- net at D5.2 (A): now also MX11.2
- net at D16.2 (A): now also MX2.2
- net at D7.2 (A): now also MX13.2
- net at D3.2 (A): now also MX18.2
- net at D12.2 (A): now also MX8.2
- net at D15.2 (A): now also MX1.2
- net at D10.2 (A): now also MX6.2
- net at D17.2 (A): now also MX3.2
- net at D19.2 (A): now also MX5.2
- net at D6.2 (A): now also MX12.2
