File: Torturous/he.kicad_sch (KiCad schematic)
At the start: 4 parts, among them J3 Conn_01x08_Pin, J5 Conn_01x05_Pin

Commit message: started the phys layout
Parts:
- J3: footprint (none) -> Connector_FFC-FPC:Hirose_FH12-8S-0.5SH_1x08-1MP_P0.50mm_Horizontal
- J5: footprint (none) -> Connector_FFC-FPC:Amphenol_F32Q-1A7x1-11005_1x05-1MP_P0.5mm_Horizontal
- S2: footprint 463091370402:463091370402 -> Microswith:463091370402
Changed lines of the file:
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@@
 			)
 		)
-		(property "Footprint" ""
+		(property "Footprint" "Connector_FFC-FPC:Hirose_FH12-8S-0.5SH_1x08-1MP_P0.50mm_Horizontal"
 			(at 38.1 39.37 0)
 			(hide yes)
@@
 			)
 		)
-		(property "Footprint" ""
+		(property "Footprint" "Connector_FFC-FPC:Amphenol_F32Q-1A7x1-11005_1x05-1MP_P0.5mm_Horizontal"
 			(at 72.39 36.83 0)
 			(hide yes)
@@
 			)
 		)
-		(property "Footprint" "463091370402:463091370402"
+		(property "Footprint" "Microswith:463091370402"
 			(at 82.55 50.8 0)
 			(hide yes)
